Commit message: fix: align OpenArm XHand kinematics

File: public/assets/openarm-xhand1/openarm_xhand1.urdf (robot description, URDF)
Before this commit: robot openarm_xhand1, 46 links, 45 joints
Links:
- added link left_hand_index_tip
- added link left_hand_mid_tip
- added link left_hand_pinky_tip
- added link left_hand_ring_tip
- added link left_hand_thumb_rota_tip
- added link right_hand_index_tip
- added link right_hand_mid_tip
- added link right_hand_pinky_tip
- added link right_hand_ring_tip
- added link right_hand_thumb_rota_tip
Joints:
- added joint left_hand_index_rota_joint3: type fixed, parent left_hand_index_rota_link2, child left_hand_index_tip, origin xyz=0 0 0.0425 rpy=0 0 0
- added joint left_hand_mid_joint3: type fixed, parent left_hand_mid_link2, child left_hand_mid_tip, origin xyz=0 0 0.0425 rpy=0 0 0
- added joint left_hand_pinky_joint3: type fixed, parent left_hand_pinky_link2, child left_hand_pinky_tip, origin xyz=0 0 0.0425 rpy=0 0 0
- added joint left_hand_ring_joint3: type fixed, parent left_hand_ring_link2, child left_hand_ring_tip, origin xyz=0 0 0.0425 rpy=0 0 0
- added joint left_hand_thumb_rota_joint3: type fixed, parent left_hand_thumb_rota_link2, child left_hand_thumb_rota_tip, origin xyz=0 -0.0504 0 rpy=0 0 0
- added joint right_hand_index_rota_joint3: type fixed, parent right_hand_index_rota_link2, child right_hand_index_tip, origin xyz=0 0 0.0425 rpy=0 0 0
- added joint right_hand_mid_joint3: type fixed, parent right_hand_mid_link2, child right_hand_mid_tip, origin xyz=0 0 0.04211 rpy=0 0 0
- added joint right_hand_pinky_joint3: type fixed, parent right_hand_pinky_link2, child right_hand_pinky_tip, origin xyz=0 0 0.0425 rpy=0 0 0
- added joint right_hand_ring_joint3: type fixed, parent right_hand_ring_link2, child right_hand_ring_tip, origin xyz=0 0 0.0425 rpy=0 0 0
- added joint right_hand_thumb_rota_joint3: type fixed, parent right_hand_thumb_rota_link2, child right_hand_thumb_rota_tip, origin xyz=0 0.0504 0 rpy=0 0 0
- joint left_hand_index_bend_joint: axis 1 0 0 -> -1 0 0
- joint left_xhand_mount: origin xyz=0 0 -0.03 rpy=3.141592653589793 0 0 -> xyz=0 0 -0.03 rpy=3.141592653589793 0 -1.570796326794897
- joint right_hand_index_bend_joint: axis -1 0 0 -> 1 0 0
- joint right_xhand_mount: origin xyz=0 0 -0.03 rpy=3.141592653589793 0 0 -> xyz=0 0 -0.03 rpy=3.141592653589793 0 1.570796326794897
